Commit message: gazebo标定以及相机模型正常显示-2026.06.10 15：07

File: src/gz_launch/config/robots/s622/s622_handeye_gazebo.urdf.xacro (robot description, xacro)
@@ -8,8 +8,8 @@
   <xacro:include filename="../common/gazebo_ros2_control.xacro"/>
   <xacro:include filename="s622_gripper_friction.xacro"/>
-  <xacro:include filename="s622_camera_mount.xacro"/>
+  <xacro:include filename="s622_handeye_camera_mount.xacro"/>
   <xacro:gz_common_plugins controllers_file="$(arg controllers_file)" enable_sensors="$(arg enable_camera)"/>
   <xacro:if value="$(arg enable_camera)">
-    <xacro:s622_gazebo_camera/>
+    <xacro:s622_gazebo_handeye_camera/>
   </xacro:if>
   <xacro:s622_gripper_friction/>

File: src/robot_model/s622_moveit_descriptions/urdf/camera/_d435.urdf.xacro (robot description, xacro)
@@ -63,9 +63,11 @@
       <visual>
         <xacro:if value="${use_mesh}">
-          <!-- the mesh origin is at front plate in between the two infrared camera axes -->
           <origin xyz="${d435_zero_depth_to_glass + d435_glass_to_front} ${-d435_cam_depth_py} 0" rpy="${M_PI/2} 0 ${M_PI/2}"/>
           <geometry>
-            <mesh filename="file://$(find realsense2_description)/meshes/d435.glb" />
+            <mesh filename="package://s622_moveit_descriptions/meshes/d435.stl" />
           </geometry>
+          <material name="DarkGrey">
+            <color rgba="0.16 0.16 0.16 1.0"/>
+          </material>
         </xacro:if>
         <xacro:unless value="${use_mesh}">

File: src/robot_model/s622_moveit_descriptions/urdf/camera/camera.xacro (robot description, xacro)
@@ -3,6 +3,6 @@
 	<!-- =========================1) RealSense D435 的 URDF 结构========================= -->
 	<!-- 用 Intel realsense2_description 提供的 D435 URDF 宏 -->
-  	<xacro:include filename="$(find realsense2_description)/urdf/_d435.urdf.xacro" />
-	<!-- <xacro:include filename="$(find s622_moveit_descriptions)/urdf/camera/_d435.urdf.xacro" /> -->
+<!-- <xacro:include filename="$(find realsense2_description)/urdf/_d435.urdf.xacro" /> -->
+	<xacro:include filename="$(find s622_moveit_descriptions)/urdf/camera/_d435.urdf.xacro" />
 	<!-- 用 Intel realsense2_description 提供的 D435 URDF 宏 -->
 	<!-- =========================2) RealSense D435 的 Gazebo 传感器定义========================= -->
@@ -53,8 +53,5 @@
             image_width="640"
             image_height="480"/>
-        <!-- camera_link 材质 -->
-        <gazebo reference="camera_link">
-            <material>Gazebo/Grey</material>
-        </gazebo>
+        <!-- camera_link 材质：使用 URDF visual 自带的材质，不强制覆盖 -->
     </xacro:macro>
 	<!-- <gazebo reference="camera_link">
