Commit message: 2026 06.16 17:26

File: src/gazebo_launch/config/robots/s622/s622_camera_mount.xacro (robot description, xacro)
@@ -2,10 +2,13 @@
 <robot xmlns:xacro="http://www.ros.org/wiki/xacro">
   <xacro:include filename="$(find s622_moveit_descriptions)/urdf/camera/camera.xacro"/>
-  <xacro:macro name="s622_gazebo_camera">
+  <xacro:macro name="s622_gazebo_camera" params="camera_fps:=60 camera_image_width:=640 camera_image_height:=480">
     <xacro:property name="PI" value="3.14159274"/>
     <xacro:camera_v0 parent="base_link">
       <origin xyz="0.25 0.7 1.0" rpy="0 ${79*PI/180} ${-PI/2}"/>
     </xacro:camera_v0>
-    <xacro:camera_gazebo_v0/>
+    <xacro:camera_gazebo_v0
+      fps="${camera_fps}"
+      image_width="${camera_image_width}"
+      image_height="${camera_image_height}"/>
   </xacro:macro>
 </robot>

File: src/gazebo_launch/config/robots/s622/s622_gazebo.urdf.xacro (robot description, xacro)
@@ -4,4 +4,7 @@
   <xacro:arg name="controllers_file" default="$(find s622_moveit_config)/config/ros2_controllers_gazebo_velocity.yaml"/>
   <xacro:arg name="enable_camera" default="true"/>
+  <xacro:arg name="camera_fps" default="60"/>
+  <xacro:arg name="camera_image_width" default="640"/>
+  <xacro:arg name="camera_image_height" default="480"/>
   <xacro:include filename="$(find s622_moveit_descriptions)/urdf/s622_moveit_descriptions.urdf"/>
   <xacro:include filename="../common/gazebo_plugins.xacro"/>
@@ -11,5 +14,8 @@
   <xacro:gz_common_plugins controllers_file="$(arg controllers_file)" enable_sensors="$(arg enable_camera)"/>
   <xacro:if value="$(arg enable_camera)">
-    <xacro:s622_gazebo_camera/>
+    <xacro:s622_gazebo_camera
+      camera_fps="$(arg camera_fps)"
+      camera_image_width="$(arg camera_image_width)"
+      camera_image_height="$(arg camera_image_height)"/>
   </xacro:if>
   <xacro:s622_gripper_friction/>

File: src/gazebo_launch/config/robots/s622/s622_handeye_camera_mount.xacro (robot description, xacro)
@@ -2,5 +2,5 @@
 <robot xmlns:xacro="http://www.ros.org/wiki/xacro">
   <xacro:include filename="$(find s622_moveit_descriptions)/urdf/camera/camera.xacro"/>
-  <xacro:macro name="s622_gazebo_handeye_camera">
+  <xacro:macro name="s622_gazebo_handeye_camera" params="camera_fps:=30 camera_image_width:=1280 camera_image_height:=720">
     <!--
       Gazebo calibration profile uses a clean eye-in-hand visual mount instead
@@ -12,5 +12,8 @@
               rpy="0 -1.57079632679 -1.57079632679"/>
     </xacro:camera_v0>
-    <xacro:camera_gazebo_v0/>
+    <xacro:camera_gazebo_v0
+      fps="${camera_fps}"
+      image_width="${camera_image_width}"
+      image_height="${camera_image_height}"/>
   </xacro:macro>
 </robot>

File: src/gazebo_launch/config/robots/s622/s622_handeye_gazebo.urdf.xacro (robot description, xacro)
@@ -4,4 +4,7 @@
   <xacro:arg name="controllers_file" default="$(find s622_moveit_config)/config/ros2_controllers_gazebo_velocity.yaml"/>
   <xacro:arg name="enable_camera" default="true"/>
+  <xacro:arg name="camera_fps" default="30"/>
+  <xacro:arg name="camera_image_width" default="1280"/>
+  <xacro:arg name="camera_image_height" default="720"/>
   <xacro:include filename="$(find s622_moveit_descriptions)/urdf/s622_moveit_descriptions.urdf"/>
   <xacro:include filename="../common/gazebo_plugins.xacro"/>
@@ -11,5 +14,8 @@
   <xacro:gz_common_plugins controllers_file="$(arg controllers_file)" enable_sensors="$(arg enable_camera)"/>
   <xacro:if value="$(arg enable_camera)">
-    <xacro:s622_gazebo_handeye_camera/>
+    <xacro:s622_gazebo_handeye_camera
+      camera_fps="$(arg camera_fps)"
+      camera_image_width="$(arg camera_image_width)"
+      camera_image_height="$(arg camera_image_height)"/>
   </xacro:if>
   <xacro:s622_gripper_friction/>

File: src/robot_model/s622_moveit_descriptions/urdf/camera/camera.xacro (robot description, xacro)
@@ -44,5 +44,5 @@
 	</xacro:macro>
 	<!-- =========================================================宏 2：Gazebo 中的相机传感器 / 材质========================================================= -->
-	<xacro:macro name="camera_gazebo_v0">
+	<xacro:macro name="camera_gazebo_v0" params="fps:=60 image_width:=640 image_height:=480">
         <!-- Gazebo 侧 D435 相机 -->
         <xacro:gazebo_d435
@@ -50,7 +50,7 @@
             gz_topic_name="camera"
             type="rgbd"
-            fps="60"
-            image_width="640"
-            image_height="480"/>
+            fps="${fps}"
+            image_width="${image_width}"
+            image_height="${image_height}"/>
         <!-- camera_link 材质：使用 URDF visual 自带的材质，不强制覆盖 -->
     </xacro:macro>
