Commit message: llm-yolo-control-2026 07.21:57

File: src/gazebo_launch/config/scenes/box.urdf (robot description, URDF)
Before this commit: robot woodenblock, 1 links, 0 joints
Links:
- removed link box
- added link base_link, mass 1.0; collision box size=0.2 0.2 0.01; visual box size=0.2 0.2 0.01
- added link wall_back, mass 0.5; collision box size=0.20 0.01 0.10; visual box size=0.20 0.01 0.10
- added link wall_front, mass 0.5; collision box size=0.2 0.01 0.1; visual box size=0.2 0.01 0.10
- added link wall_left, mass 0.5; collision box size=0.01 0.20 0.10; visual box size=0.01 0.20 0.10
- added link wall_right, mass 0.5; collision box size=0.01 0.20 0.10; visual box size=0.01 0.20 0.10
Joints:
- added joint joint_back: type fixed, parent base_link, child wall_back, origin xyz=0 0.1 0.05 rpy=0 0 0
- added joint joint_front: type fixed, parent base_link, child wall_front, origin xyz=0 -0.1 0.05 rpy=0 0 0
- added joint joint_left: type fixed, parent base_link, child wall_left, origin xyz=-0.1 0 0.05 rpy=0 0 0
- added joint joint_right: type fixed, parent base_link, child wall_right, origin xyz=0.1 0 0.05 rpy=0 0 0
