Commit message: 2026 0804 2137 -标定模块化收敛

File: src/gazebo_launch/config/robots/fairino_arm/fairino_arm_handeye_camera_mount.xacro (robot description, xacro)
@@ -9,5 +9,5 @@
     -->
     <xacro:camera_v0 parent="grasp_frame">
-      <origin xyz="0.000 -0.0375 -0.060"
+      <origin xyz="0.000 -0.0475 -0.060"
               rpy="0 -1.57079632679 -1.57079632679"/>
     </xacro:camera_v0>
