Commit message: 2026.08.02 1400-相机仿真内参的构建

File: src/camera_ws/realsense2_gz_description/urdf/_d435.gazebo.xacro (robot description, xacro)
@@ -21,16 +21,24 @@
   image_width:=1280
   image_height:=720
+  fx:=0 fy:=0 cx:=0 cy:=0
+  k1:=0 k2:=0 k3:=0 p1:=0 p2:=0
+  noise_stddev:=0
+  h_fov:=1.2042771838760873
+  v_fov:=0.7330382858376184
+  depth_image_width:=1280
+  depth_image_height:=720
+  depth_fx:=0 depth_fy:=0 depth_cx:=0 depth_cy:=0
+  depth_k1:=0 depth_k2:=0 depth_k3:=0 depth_p1:=0 depth_p2:=0
+  depth_h_fov:=1.5184364492350666
+  depth_v_fov:=1.0122909661567112
+  depth_near_m:=0.28
+  depth_far_m:=3.0
   triggered:=false">
     <!-- Realsense D435 RGB properties
     Assumptions:
     Parent system (URDF or sdf) will start the Gazebo Sensors plugin. See notes in the camera.gazebo.xacros.
-    Simulated RGB and Depth sensors are in the same location as the RGB sensor of the physical camera.
-    Simulated RGB and Depth sensors and have the same FOV as the RGB physical sensor.
-    Note: physical hardware publishes pointcloud in `camera_depth_optical_frame` where this sensor will use
-    the referenced camera color_frame. -->
-    <xacro:property name="realsense_h_fov" value="${69 * pi/180}" />
-    <xacro:property name="realsense_v_fov" value="${42 * pi/180}" />
-    <xacro:property name="min_depth" value="0.28" />
-    <xacro:property name="max_depth" value="3.0" />
+    The RGBD sensor remains colocated with the physical RGB camera and
+    produces the ideal aligned-depth stream. A separate depth_camera below
+    provides the native depth resolution and intrinsics at camera_depth_frame. -->
     <xacro:if value="${type == 'rgbd'}">
         <xacro:gazebo_rgbd name="${name}"
@@ -39,8 +47,22 @@
                            image_width="${image_width}"
                            image_height="${image_height}"
-                           h_fov="${realsense_h_fov}"
-                           v_fov="${realsense_v_fov}"
-                           min_depth="${min_depth}"
-                           max_depth="${max_depth}"/>
+                           fx="${fx}" fy="${fy}" cx="${cx}" cy="${cy}"
+                           k1="${k1}" k2="${k2}" k3="${k3}" p1="${p1}" p2="${p2}"
+                           noise_stddev="${noise_stddev}"
+                           h_fov="${h_fov}"
+                           v_fov="${v_fov}"
+                           min_depth="${depth_near_m}"
+                           max_depth="${depth_far_m}"/>
+        <xacro:gazebo_depth_camera name="${name}"
+                                   fps="${fps}"
+                                   gz_topic_name="${gz_topic_name}/native_depth/image"
+                                   image_width="${depth_image_width}"
+                                   image_height="${depth_image_height}"
+                                   fx="${depth_fx}" fy="${depth_fy}" cx="${depth_cx}" cy="${depth_cy}"
+                                   k1="${depth_k1}" k2="${depth_k2}" k3="${depth_k3}" p1="${depth_p1}" p2="${depth_p2}"
+                                   h_fov="${depth_h_fov}"
+                                   v_fov="${depth_v_fov}"
+                                   min_depth="${depth_near_m}"
+                                   max_depth="${depth_far_m}"/>
     </xacro:if>
     <xacro:if value="${type == 'rgb'}">
@@ -50,6 +72,6 @@
                         image_width="${image_width}"
                         image_height="${image_height}"
-                        h_fov="${realsense_h_fov}"
-                        v_fov="${realsense_v_fov}"
+                        h_fov="${h_fov}"
+                        v_fov="${v_fov}"
                         triggered="${triggered}"/>
     </xacro:if>

File: src/camera_ws/realsense2_gz_description/urdf/rgbd_camera.gazebo.xacro (robot description, xacro)
@@ -19,4 +19,7 @@
   image_width:=1280
   image_height:=720
+  fx:=0 fy:=0 cx:=0 cy:=0
+  k1:=0 k2:=0 k3:=0 p1:=0 p2:=0
+  noise_stddev:=0
   h_fov
   v_fov
@@ -29,8 +32,10 @@
     Note: physical hardware publishes pointcloud in `camera_depth_optical_frame` where this sensor will use
     the referenced camera color_frame. -->
-    <xacro:property name="fx" value="${image_width * 0.5 / tan(h_fov * 0.5)}" />
-    <xacro:property name="fy" value="${image_height * 0.5 / tan(v_fov * 0.5)}" />
-    <xacro:property name="cx" value="${image_width * 0.5}" />
-    <xacro:property name="cy" value="${image_height * 0.5}" />
+    <xacro:property name="computed_fx" value="${image_width * 0.5 / tan(h_fov * 0.5)}" />
+    <xacro:property name="computed_fy" value="${image_height * 0.5 / tan(v_fov * 0.5)}" />
+    <xacro:property name="effective_fx" value="${fx if fx > 0 else computed_fx}" />
+    <xacro:property name="effective_fy" value="${fy if fy > 0 else computed_fy}" />
+    <xacro:property name="effective_cx" value="${cx if cx > 0 else image_width * 0.5}" />
+    <xacro:property name="effective_cy" value="${cy if cy > 0 else image_height * 0.5}" />
     <!-- <xacro:property name="min_depth" value="0.52" />
     <xacro:property name="max_depth" value="6.0" /> -->
@@ -49,24 +54,24 @@
                 </clip>
                 <distortion>
-                    <k1>0.0</k1>
-                    <k2>0.0</k2>
-                    <k3>0.0</k3>
-                    <p1>0.0</p1>
-                    <p2>0.0</p2>
+                    <k1>${k1}</k1>
+                    <k2>${k2}</k2>
+                    <k3>${k3}</k3>
+                    <p1>${p1}</p1>
+                    <p2>${p2}</p2>
                     <center>0.5 0.5</center>
                 </distortion>
                 <lens>
                     <intrinsics>
-                        <fx>${fx}</fx>
-                        <fy>${fy}</fy>
-                        <cx>${cx}</cx>
-                        <cy>${cy}</cy>
+                        <fx>${effective_fx}</fx>
+                        <fy>${effective_fy}</fy>
+                        <cx>${effective_cx}</cx>
+                        <cy>${effective_cy}</cy>
                         <s>0</s>
                     </intrinsics>
                     <projection>
-                        <p_fx>${fx}</p_fx>
-                        <p_fy>${fy}</p_fy>
-                        <p_cx>${cx}</p_cx>
-                        <p_cy>${cy}</p_cy>
+                        <p_fx>${effective_fx}</p_fx>
+                        <p_fy>${effective_fy}</p_fy>
+                        <p_cx>${effective_cx}</p_cx>
+                        <p_cy>${effective_cy}</p_cy>
                         <tx>0</tx>
                         <ty>0</ty>
@@ -76,5 +81,5 @@
                     <type>gaussian</type>
                     <mean>0</mean>
-                    <stddev>0.00</stddev>
+                    <stddev>${noise_stddev}</stddev>
                 </noise>
                 <depth_camera>
@@ -95,3 +100,75 @@
     </gazebo>
 </xacro:macro>
+<!--
+  A native D435 depth stream.  This intentionally models only the depth
+  camera's independently calibrated image geometry; it does not create the
+  two IR streams or simulate the D4 stereo pipeline.
+-->
+<xacro:macro name="gazebo_depth_camera" params="
+  name:=camera
+  fps:=15
+  gz_topic_name:=camera/native_depth/image
+  image_width:=1280
+  image_height:=720
+  fx:=0 fy:=0 cx:=0 cy:=0
+  k1:=0 k2:=0 k3:=0 p1:=0 p2:=0
+  h_fov
+  v_fov
+  min_depth
+  max_depth">
+    <xacro:property name="computed_fx" value="${image_width * 0.5 / tan(h_fov * 0.5)}" />
+    <xacro:property name="computed_fy" value="${image_height * 0.5 / tan(v_fov * 0.5)}" />
+    <xacro:property name="effective_fx" value="${fx if fx > 0 else computed_fx}" />
+    <xacro:property name="effective_fy" value="${fy if fy > 0 else computed_fy}" />
+    <xacro:property name="effective_cx" value="${cx if cx > 0 else image_width * 0.5}" />
+    <xacro:property name="effective_cy" value="${cy if cy > 0 else image_height * 0.5}" />
+    <gazebo reference="${name}_depth_frame">
+        <sensor name="${name}_native_depth" type="depth_camera">
+            <camera>
+                <horizontal_fov>${h_fov}</horizontal_fov>
+                <image>
+                    <width>${image_width}</width>
+                    <height>${image_height}</height>
+                    <format>R_FLOAT32</format>
+                </image>
+                <clip>
+                    <near>${min_depth}</near>
+                    <far>${max_depth}</far>
+                </clip>
+                <distortion>
+                    <k1>${k1}</k1>
+                    <k2>${k2}</k2>
+                    <k3>${k3}</k3>
+                    <p1>${p1}</p1>
+                    <p2>${p2}</p2>
+                    <center>0.5 0.5</center>
+                </distortion>
+                <lens>
+                    <intrinsics>
+                        <fx>${effective_fx}</fx>
+                        <fy>${effective_fy}</fy>
+                        <cx>${effective_cx}</cx>
+                        <cy>${effective_cy}</cy>
+                        <s>0</s>
+                    </intrinsics>
+                    <projection>
+                        <p_fx>${effective_fx}</p_fx>
+                        <p_fy>${effective_fy}</p_fy>
+                        <p_cx>${effective_cx}</p_cx>
+                        <p_cy>${effective_cy}</p_cy>
+                        <tx>0</tx>
+                        <ty>0</ty>
+                    </projection>
+                </lens>
+                <optical_frame_id>${name}_depth_optical_frame</optical_frame_id>
+            </camera>
+            <ignition_frame_id>${name}_depth_frame</ignition_frame_id>
+            <always_on>1</always_on>
+            <update_rate>${fps}</update_rate>
+            <visualize>false</visualize>
+            <topic>${gz_topic_name}</topic>
+            <enable_metrics>false</enable_metrics>
+        </sensor>
+    </gazebo>
+</xacro:macro>
 </robot>

File: src/fairino_robot_support/fairino_arm_moveit_descriptions/urdf/camera/camera.xacro (robot description, xacro)
@@ -44,5 +44,5 @@
 	</xacro:macro>
 	<!-- =========================================================宏 2：Gazebo 中的相机传感器 / 材质========================================================= -->
-	<xacro:macro name="camera_gazebo_v0" params="fps:=60 image_width:=640 image_height:=480">
+	<xacro:macro name="camera_gazebo_v0" params="fps:=60 image_width:=640 image_height:=480 fx:=0 fy:=0 cx:=0 cy:=0 k1:=0 k2:=0 k3:=0 p1:=0 p2:=0 noise_stddev:=0 h_fov:=1.2042771838760873 v_fov:=0.7330382858376184 depth_image_width:=1280 depth_image_height:=720 depth_fx:=0 depth_fy:=0 depth_cx:=0 depth_cy:=0 depth_k1:=0 depth_k2:=0 depth_k3:=0 depth_p1:=0 depth_p2:=0 depth_h_fov:=1.5184364492350666 depth_v_fov:=1.0122909661567112 depth_near_m:=0.28 depth_far_m:=3.0">
         <!-- Gazebo 侧 D435 相机 -->
         <xacro:gazebo_d435
@@ -52,5 +52,15 @@
             fps="${fps}"
             image_width="${image_width}"
-            image_height="${image_height}"/>
+            image_height="${image_height}"
+            fx="${fx}" fy="${fy}" cx="${cx}" cy="${cy}"
+            k1="${k1}" k2="${k2}" k3="${k3}" p1="${p1}" p2="${p2}"
+            noise_stddev="${noise_stddev}"
+            h_fov="${h_fov}" v_fov="${v_fov}"
+            depth_image_width="${depth_image_width}"
+            depth_image_height="${depth_image_height}"
+            depth_fx="${depth_fx}" depth_fy="${depth_fy}" depth_cx="${depth_cx}" depth_cy="${depth_cy}"
+            depth_k1="${depth_k1}" depth_k2="${depth_k2}" depth_k3="${depth_k3}" depth_p1="${depth_p1}" depth_p2="${depth_p2}"
+            depth_h_fov="${depth_h_fov}" depth_v_fov="${depth_v_fov}"
+            depth_near_m="${depth_near_m}" depth_far_m="${depth_far_m}"/>
         <!-- camera_link 材质：使用 URDF visual 自带的材质，不强制覆盖 -->
     </xacro:macro>

File: src/gazebo_launch/config/robots/fairino_arm/fairino_arm_camera_mount.xacro (robot description, xacro)
@@ -2,5 +2,5 @@
 <robot xmlns:xacro="http://www.ros.org/wiki/xacro">
   <xacro:include filename="$(find fairino_arm_moveit_descriptions)/urdf/camera/camera.xacro"/>
-  <xacro:macro name="fairino_arm_gazebo_camera" params="camera_fps:=60 camera_image_width:=640 camera_image_height:=480">
+  <xacro:macro name="fairino_arm_gazebo_camera" params="camera_fps:=60 camera_image_width:=640 camera_image_height:=480 camera_fx:=0 camera_fy:=0 camera_cx:=0 camera_cy:=0 camera_k1:=0 camera_k2:=0 camera_k3:=0 camera_p1:=0 camera_p2:=0 camera_noise_stddev:=0 camera_h_fov:=1.2042771838760873 camera_v_fov:=0.7330382858376184 camera_depth_image_width:=1280 camera_depth_image_height:=720 camera_depth_fx:=0 camera_depth_fy:=0 camera_depth_cx:=0 camera_depth_cy:=0 camera_depth_k1:=0 camera_depth_k2:=0 camera_depth_k3:=0 camera_depth_p1:=0 camera_depth_p2:=0 camera_depth_h_fov:=1.5184364492350666 camera_depth_v_fov:=1.0122909661567112 camera_depth_near_m:=0.28 camera_depth_far_m:=3.0">
     <xacro:property name="PI" value="3.14159274"/>
     <xacro:camera_v0 parent="base_link">
@@ -10,5 +10,15 @@
       fps="${camera_fps}"
       image_width="${camera_image_width}"
-      image_height="${camera_image_height}"/>
+      image_height="${camera_image_height}"
+      fx="${camera_fx}" fy="${camera_fy}" cx="${camera_cx}" cy="${camera_cy}"
+      k1="${camera_k1}" k2="${camera_k2}" k3="${camera_k3}" p1="${camera_p1}" p2="${camera_p2}"
+      noise_stddev="${camera_noise_stddev}"
+      h_fov="${camera_h_fov}" v_fov="${camera_v_fov}"
+      depth_image_width="${camera_depth_image_width}"
+      depth_image_height="${camera_depth_image_height}"
+      depth_fx="${camera_depth_fx}" depth_fy="${camera_depth_fy}" depth_cx="${camera_depth_cx}" depth_cy="${camera_depth_cy}"
+      depth_k1="${camera_depth_k1}" depth_k2="${camera_depth_k2}" depth_k3="${camera_depth_k3}" depth_p1="${camera_depth_p1}" depth_p2="${camera_depth_p2}"
+      depth_h_fov="${camera_depth_h_fov}" depth_v_fov="${camera_depth_v_fov}"
+      depth_near_m="${camera_depth_near_m}" depth_far_m="${camera_depth_far_m}"/>
   </xacro:macro>
 </robot>

File: src/gazebo_launch/config/robots/fairino_arm/fairino_arm_gazebo.urdf.xacro (robot description, xacro)
@@ -7,4 +7,20 @@
   <xacro:arg name="camera_image_width" default="640"/>
   <xacro:arg name="camera_image_height" default="480"/>
+  <xacro:arg name="camera_fx" default="0"/><xacro:arg name="camera_fy" default="0"/>
+  <xacro:arg name="camera_cx" default="0"/><xacro:arg name="camera_cy" default="0"/>
+  <xacro:arg name="camera_k1" default="0"/><xacro:arg name="camera_k2" default="0"/><xacro:arg name="camera_k3" default="0"/>
+  <xacro:arg name="camera_p1" default="0"/><xacro:arg name="camera_p2" default="0"/><xacro:arg name="camera_noise_stddev" default="0"/>
+  <xacro:arg name="camera_h_fov" default="1.2042771838760873"/>
+  <xacro:arg name="camera_v_fov" default="0.7330382858376184"/>
+  <xacro:arg name="camera_depth_image_width" default="1280"/>
+  <xacro:arg name="camera_depth_image_height" default="720"/>
+  <xacro:arg name="camera_depth_fx" default="0"/><xacro:arg name="camera_depth_fy" default="0"/>
+  <xacro:arg name="camera_depth_cx" default="0"/><xacro:arg name="camera_depth_cy" default="0"/>
+  <xacro:arg name="camera_depth_k1" default="0"/><xacro:arg name="camera_depth_k2" default="0"/><xacro:arg name="camera_depth_k3" default="0"/>
+  <xacro:arg name="camera_depth_p1" default="0"/><xacro:arg name="camera_depth_p2" default="0"/>
+  <xacro:arg name="camera_depth_h_fov" default="1.5184364492350666"/>
+  <xacro:arg name="camera_depth_v_fov" default="1.0122909661567112"/>
+  <xacro:arg name="camera_depth_near_m" default="0.28"/>
+  <xacro:arg name="camera_depth_far_m" default="3.0"/>
   <xacro:include filename="$(find fairino_arm_moveit_descriptions)/urdf/fairino_arm_moveit_descriptions.urdf"/>
   <xacro:include filename="../common/gazebo_plugins.xacro"/>
@@ -17,5 +33,15 @@
       camera_fps="$(arg camera_fps)"
       camera_image_width="$(arg camera_image_width)"
-      camera_image_height="$(arg camera_image_height)"/>
+      camera_image_height="$(arg camera_image_height)"
+      camera_fx="$(arg camera_fx)" camera_fy="$(arg camera_fy)" camera_cx="$(arg camera_cx)" camera_cy="$(arg camera_cy)"
+      camera_k1="$(arg camera_k1)" camera_k2="$(arg camera_k2)" camera_k3="$(arg camera_k3)" camera_p1="$(arg camera_p1)" camera_p2="$(arg camera_p2)"
+      camera_noise_stddev="$(arg camera_noise_stddev)"
+      camera_h_fov="$(arg camera_h_fov)" camera_v_fov="$(arg camera_v_fov)"
+      camera_depth_image_width="$(arg camera_depth_image_width)"
+      camera_depth_image_height="$(arg camera_depth_image_height)"
+      camera_depth_fx="$(arg camera_depth_fx)" camera_depth_fy="$(arg camera_depth_fy)" camera_depth_cx="$(arg camera_depth_cx)" camera_depth_cy="$(arg camera_depth_cy)"
+      camera_depth_k1="$(arg camera_depth_k1)" camera_depth_k2="$(arg camera_depth_k2)" camera_depth_k3="$(arg camera_depth_k3)" camera_depth_p1="$(arg camera_depth_p1)" camera_depth_p2="$(arg camera_depth_p2)"
+      camera_depth_h_fov="$(arg camera_depth_h_fov)" camera_depth_v_fov="$(arg camera_depth_v_fov)"
+      camera_depth_near_m="$(arg camera_depth_near_m)" camera_depth_far_m="$(arg camera_depth_far_m)"/>
   </xacro:if>
   <xacro:fairino_arm_gripper_friction/>

File: src/gazebo_launch/config/robots/fairino_arm/fairino_arm_handeye_camera_mount.xacro (robot description, xacro)
@@ -2,5 +2,5 @@
 <robot xmlns:xacro="http://www.ros.org/wiki/xacro">
   <xacro:include filename="$(find fairino_arm_moveit_descriptions)/urdf/camera/camera.xacro"/>
-  <xacro:macro name="fairino_arm_gazebo_handeye_camera" params="camera_fps:=30 camera_image_width:=1280 camera_image_height:=720">
+  <xacro:macro name="fairino_arm_gazebo_handeye_camera" params="camera_fps:=30 camera_image_width:=1280 camera_image_height:=720 camera_fx:=0 camera_fy:=0 camera_cx:=0 camera_cy:=0 camera_k1:=0 camera_k2:=0 camera_k3:=0 camera_p1:=0 camera_p2:=0 camera_noise_stddev:=0 camera_h_fov:=1.2042771838760873 camera_v_fov:=0.7330382858376184 camera_depth_image_width:=1280 camera_depth_image_height:=720 camera_depth_fx:=0 camera_depth_fy:=0 camera_depth_cx:=0 camera_depth_cy:=0 camera_depth_k1:=0 camera_depth_k2:=0 camera_depth_k3:=0 camera_depth_p1:=0 camera_depth_p2:=0 camera_depth_h_fov:=1.5184364492350666 camera_depth_v_fov:=1.0122909661567112 camera_depth_near_m:=0.28 camera_depth_far_m:=3.0">
     <!--
       Gazebo calibration profile uses a clean eye-in-hand visual mount instead
@@ -15,5 +15,15 @@
       fps="${camera_fps}"
       image_width="${camera_image_width}"
-      image_height="${camera_image_height}"/>
+      image_height="${camera_image_height}"
+      fx="${camera_fx}" fy="${camera_fy}" cx="${camera_cx}" cy="${camera_cy}"
+      k1="${camera_k1}" k2="${camera_k2}" k3="${camera_k3}" p1="${camera_p1}" p2="${camera_p2}"
+      noise_stddev="${camera_noise_stddev}"
+      h_fov="${camera_h_fov}" v_fov="${camera_v_fov}"
+      depth_image_width="${camera_depth_image_width}"
+      depth_image_height="${camera_depth_image_height}"
+      depth_fx="${camera_depth_fx}" depth_fy="${camera_depth_fy}" depth_cx="${camera_depth_cx}" depth_cy="${camera_depth_cy}"
+      depth_k1="${camera_depth_k1}" depth_k2="${camera_depth_k2}" depth_k3="${camera_depth_k3}" depth_p1="${camera_depth_p1}" depth_p2="${camera_depth_p2}"
+      depth_h_fov="${camera_depth_h_fov}" depth_v_fov="${camera_depth_v_fov}"
+      depth_near_m="${camera_depth_near_m}" depth_far_m="${camera_depth_far_m}"/>
   </xacro:macro>
 </robot>

File: src/gazebo_launch/config/robots/fairino_arm/fairino_arm_handeye_gazebo.urdf.xacro (robot description, xacro)
@@ -7,4 +7,20 @@
   <xacro:arg name="camera_image_width" default="1280"/>
   <xacro:arg name="camera_image_height" default="720"/>
+  <xacro:arg name="camera_fx" default="0"/><xacro:arg name="camera_fy" default="0"/>
+  <xacro:arg name="camera_cx" default="0"/><xacro:arg name="camera_cy" default="0"/>
+  <xacro:arg name="camera_k1" default="0"/><xacro:arg name="camera_k2" default="0"/><xacro:arg name="camera_k3" default="0"/>
+  <xacro:arg name="camera_p1" default="0"/><xacro:arg name="camera_p2" default="0"/><xacro:arg name="camera_noise_stddev" default="0"/>
+  <xacro:arg name="camera_h_fov" default="1.2042771838760873"/>
+  <xacro:arg name="camera_v_fov" default="0.7330382858376184"/>
+  <xacro:arg name="camera_depth_image_width" default="1280"/>
+  <xacro:arg name="camera_depth_image_height" default="720"/>
+  <xacro:arg name="camera_depth_fx" default="0"/><xacro:arg name="camera_depth_fy" default="0"/>
+  <xacro:arg name="camera_depth_cx" default="0"/><xacro:arg name="camera_depth_cy" default="0"/>
+  <xacro:arg name="camera_depth_k1" default="0"/><xacro:arg name="camera_depth_k2" default="0"/><xacro:arg name="camera_depth_k3" default="0"/>
+  <xacro:arg name="camera_depth_p1" default="0"/><xacro:arg name="camera_depth_p2" default="0"/>
+  <xacro:arg name="camera_depth_h_fov" default="1.5184364492350666"/>
+  <xacro:arg name="camera_depth_v_fov" default="1.0122909661567112"/>
+  <xacro:arg name="camera_depth_near_m" default="0.28"/>
+  <xacro:arg name="camera_depth_far_m" default="3.0"/>
   <xacro:include filename="$(find fairino_arm_moveit_descriptions)/urdf/fairino_arm_moveit_descriptions.urdf"/>
   <xacro:include filename="../common/gazebo_plugins.xacro"/>
@@ -17,5 +33,15 @@
       camera_fps="$(arg camera_fps)"
       camera_image_width="$(arg camera_image_width)"
-      camera_image_height="$(arg camera_image_height)"/>
+      camera_image_height="$(arg camera_image_height)"
+      camera_fx="$(arg camera_fx)" camera_fy="$(arg camera_fy)" camera_cx="$(arg camera_cx)" camera_cy="$(arg camera_cy)"
+      camera_k1="$(arg camera_k1)" camera_k2="$(arg camera_k2)" camera_k3="$(arg camera_k3)" camera_p1="$(arg camera_p1)" camera_p2="$(arg camera_p2)"
+      camera_noise_stddev="$(arg camera_noise_stddev)"
+      camera_h_fov="$(arg camera_h_fov)" camera_v_fov="$(arg camera_v_fov)"
+      camera_depth_image_width="$(arg camera_depth_image_width)"
+      camera_depth_image_height="$(arg camera_depth_image_height)"
+      camera_depth_fx="$(arg camera_depth_fx)" camera_depth_fy="$(arg camera_depth_fy)" camera_depth_cx="$(arg camera_depth_cx)" camera_depth_cy="$(arg camera_depth_cy)"
+      camera_depth_k1="$(arg camera_depth_k1)" camera_depth_k2="$(arg camera_depth_k2)" camera_depth_k3="$(arg camera_depth_k3)" camera_depth_p1="$(arg camera_depth_p1)" camera_depth_p2="$(arg camera_depth_p2)"
+      camera_depth_h_fov="$(arg camera_depth_h_fov)" camera_depth_v_fov="$(arg camera_depth_v_fov)"
+      camera_depth_near_m="$(arg camera_depth_near_m)" camera_depth_far_m="$(arg camera_depth_far_m)"/>
   </xacro:if>
   <xacro:fairino_arm_gripper_friction/>
