Commit message: 2026 08.09 -手眼标定的优化

File: src/camera_ws/realsense2_gz_description/urdf/_d435.gazebo.xacro (robot description, xacro)
@@ -54,15 +54,4 @@
                            min_depth="${depth_near_m}"
                            max_depth="${depth_far_m}"/>
-        <xacro:gazebo_depth_camera name="${name}"
-                                   fps="${fps}"
-                                   gz_topic_name="${gz_topic_name}/native_depth/image"
-                                   image_width="${depth_image_width}"
-                                   image_height="${depth_image_height}"
-                                   fx="${depth_fx}" fy="${depth_fy}" cx="${depth_cx}" cy="${depth_cy}"
-                                   k1="${depth_k1}" k2="${depth_k2}" k3="${depth_k3}" p1="${depth_p1}" p2="${depth_p2}"
-                                   h_fov="${depth_h_fov}"
-                                   v_fov="${depth_v_fov}"
-                                   min_depth="${depth_near_m}"
-                                   max_depth="${depth_far_m}"/>
     </xacro:if>
     <xacro:if value="${type == 'rgb'}">
@@ -76,4 +65,15 @@
                         triggered="${triggered}"/>
     </xacro:if>
+    <xacro:gazebo_depth_camera name="${name}"
+                               fps="${fps}"
+                               gz_topic_name="${gz_topic_name}/native_depth/image"
+                               image_width="${depth_image_width}"
+                               image_height="${depth_image_height}"
+                               fx="${depth_fx}" fy="${depth_fy}" cx="${depth_cx}" cy="${depth_cy}"
+                               k1="${depth_k1}" k2="${depth_k2}" k3="${depth_k3}" p1="${depth_p1}" p2="${depth_p2}"
+                               h_fov="${depth_h_fov}"
+                               v_fov="${depth_v_fov}"
+                               min_depth="${depth_near_m}"
+                               max_depth="${depth_far_m}"/>
 </xacro:macro>
 </robot>

File: src/fairino_robot_support/fairino_arm_moveit_config/config/fairino_arm_moveit_descriptions.urdf.xacro (robot description, xacro)
@@ -6,4 +6,4 @@
     <!-- Import control_xacro -->
     <xacro:include filename="fairino_arm_moveit_descriptions.ros2_control.xacro" />
-    <xacro:fairino_arm_moveit_descriptions_ros2_control name="FakeSystem" initial_positions_file="$(arg initial_positions_file)"/>
+    <xacro:fairino_arm_moveit_descriptions_ros2_control name="FairinoSystem" initial_positions_file="$(arg initial_positions_file)"/>
 </robot>

File: src/fairino_robot_support/fairino_arm_moveit_descriptions/urdf/camera/camera.xacro (robot description, xacro)
@@ -44,10 +44,10 @@
 	</xacro:macro>
 	<!-- =========================================================宏 2：Gazebo 中的相机传感器 / 材质========================================================= -->
-	<xacro:macro name="camera_gazebo_v0" params="fps:=60 image_width:=640 image_height:=480 fx:=0 fy:=0 cx:=0 cy:=0 k1:=0 k2:=0 k3:=0 p1:=0 p2:=0 noise_stddev:=0 h_fov:=1.2042771838760873 v_fov:=0.7330382858376184 depth_image_width:=1280 depth_image_height:=720 depth_fx:=0 depth_fy:=0 depth_cx:=0 depth_cy:=0 depth_k1:=0 depth_k2:=0 depth_k3:=0 depth_p1:=0 depth_p2:=0 depth_h_fov:=1.5184364492350666 depth_v_fov:=1.0122909661567112 depth_near_m:=0.28 depth_far_m:=3.0">
+	<xacro:macro name="camera_gazebo_v0" params="sensor_type:=rgbd fps:=60 image_width:=640 image_height:=480 fx:=0 fy:=0 cx:=0 cy:=0 k1:=0 k2:=0 k3:=0 p1:=0 p2:=0 noise_stddev:=0 h_fov:=1.2042771838760873 v_fov:=0.7330382858376184 depth_image_width:=1280 depth_image_height:=720 depth_fx:=0 depth_fy:=0 depth_cx:=0 depth_cy:=0 depth_k1:=0 depth_k2:=0 depth_k3:=0 depth_p1:=0 depth_p2:=0 depth_h_fov:=1.5184364492350666 depth_v_fov:=1.0122909661567112 depth_near_m:=0.28 depth_far_m:=3.0">
         <!-- Gazebo 侧 D435 相机 -->
         <xacro:gazebo_d435
             name="camera"
             gz_topic_name="camera"
-            type="rgbd"
+            type="${sensor_type}"
             fps="${fps}"
             image_width="${image_width}"

File: src/gazebo_launch/config/robots/fairino_arm/fairino_arm_handeye_camera_mount.xacro (robot description, xacro)
@@ -9,8 +9,9 @@
     -->
     <xacro:camera_v0 parent="grasp_frame">
-      <origin xyz="0.000 -0.0475 -0.060"
+      <origin xyz="0.000 -0.05 -0.09"
               rpy="0 -1.57079632679 -1.57079632679"/>
     </xacro:camera_v0>
     <xacro:camera_gazebo_v0
+      sensor_type="rgb"
       fps="${camera_fps}"
       image_width="${camera_image_width}"

Commit message: 2026 08.16-删除包GraphExecuter和建立正确仿真环境rgbd相机渲染

File: src/camera_ws/realsense2_gz_description/urdf/_d435.gazebo.xacro (robot description, xacro)
@@ -14,4 +14,69 @@
              ign topic -t "/name/trigger" -m Boolean -p "data: true" -n 1
 -->
+<xacro:macro name="gazebo_aligned_depth_camera" params="
+  name:=camera
+  fps:=15
+  gz_topic_name:=camera
+  image_width:=1280
+  image_height:=720
+  fx:=0 fy:=0 cx:=0 cy:=0
+  h_fov
+  v_fov
+  min_depth
+  max_depth
+  camera_info_topic">
+    <!-- A colocated depth camera that avoids Ogre2's rgbd_camera path. -->
+    <xacro:property name="effective_fx" value="${fx if fx > 0 else image_width * 0.5 / tan(h_fov * 0.5)}" />
+    <xacro:property name="effective_fy" value="${fy if fy > 0 else image_height * 0.5 / tan(v_fov * 0.5)}" />
+    <xacro:property name="effective_cx" value="${cx if cx > 0 else image_width * 0.5}" />
+    <xacro:property name="effective_cy" value="${cy if cy > 0 else image_height * 0.5}" />
+    <gazebo reference="${name}_color_frame">
+        <sensor name="${name}_aligned_depth" type="depth_camera">
+            <camera>
+                <camera_info_topic>${camera_info_topic}</camera_info_topic>
+                <horizontal_fov>${h_fov}</horizontal_fov>
+                <lens>
+                    <intrinsics>
+                        <fx>${effective_fx}</fx>
+                        <fy>${effective_fy}</fy>
+                        <cx>${effective_cx}</cx>
+                        <cy>${effective_cy}</cy>
+                        <s>0</s>
+                    </intrinsics>
+                    <projection>
+                        <p_fx>${effective_fx}</p_fx>
+                        <p_fy>${effective_fy}</p_fy>
+                        <p_cx>${effective_cx}</p_cx>
+                        <p_cy>${effective_cy}</p_cy>
+                        <tx>0</tx>
+                        <ty>0</ty>
+                    </projection>
+                </lens>
+                <image>
+                    <width>${image_width}</width>
+                    <height>${image_height}</height>
+                    <format>R_FLOAT32</format>
+                </image>
+                <clip>
+                    <near>${min_depth}</near>
+                    <far>${max_depth}</far>
+                </clip>
+                <depth_camera>
+                    <clip>
+                        <near>${min_depth}</near>
+                        <far>${max_depth}</far>
+                    </clip>
+                </depth_camera>
+                <optical_frame_id>${name}_color_optical_frame</optical_frame_id>
+            </camera>
+            <ignition_frame_id>${name}_color_frame</ignition_frame_id>
+            <always_on>1</always_on>
+            <update_rate>${fps}</update_rate>
+            <visualize>false</visualize>
+            <topic>${gz_topic_name}/aligned_depth/image</topic>
+            <enable_metrics>false</enable_metrics>
+        </sensor>
+    </gazebo>
+</xacro:macro>
 <xacro:macro name="gazebo_d435" params="
   name:=camera
@@ -41,18 +106,4 @@
     produces the ideal aligned-depth stream. A separate depth_camera below
     provides the native depth resolution and intrinsics at camera_depth_frame. -->
-    <xacro:if value="${type == 'rgbd'}">
-        <xacro:gazebo_rgbd name="${name}"
-                           fps="${fps}"
-                           gz_topic_name="${gz_topic_name}"
-                           image_width="${image_width}"
-                           image_height="${image_height}"
-                           fx="${fx}" fy="${fy}" cx="${cx}" cy="${cy}"
-                           k1="${k1}" k2="${k2}" k3="${k3}" p1="${p1}" p2="${p2}"
-                           noise_stddev="${noise_stddev}"
-                           h_fov="${h_fov}"
-                           v_fov="${v_fov}"
-                           min_depth="${depth_near_m}"
-                           max_depth="${depth_far_m}"/>
-    </xacro:if>
     <xacro:if value="${type == 'rgb'}">
         <xacro:gazebo_rgb name="${name}"
@@ -63,17 +114,40 @@
                         h_fov="${h_fov}"
                         v_fov="${v_fov}"
-                        triggered="${triggered}"/>
+                        triggered="${triggered}"
+                        camera_info_topic="${gz_topic_name}/camera_info"/>
     </xacro:if>
-    <xacro:gazebo_depth_camera name="${name}"
-                               fps="${fps}"
-                               gz_topic_name="${gz_topic_name}/native_depth/image"
-                               image_width="${depth_image_width}"
-                               image_height="${depth_image_height}"
-                               fx="${depth_fx}" fy="${depth_fy}" cx="${depth_cx}" cy="${depth_cy}"
-                               k1="${depth_k1}" k2="${depth_k2}" k3="${depth_k3}" p1="${depth_p1}" p2="${depth_p2}"
-                               h_fov="${depth_h_fov}"
-                               v_fov="${depth_v_fov}"
-                               min_depth="${depth_near_m}"
-                               max_depth="${depth_far_m}"/>
+    <xacro:if value="${type == 'rgbd'}">
+        <xacro:gazebo_rgb name="${name}"
+                        fps="${fps}"
+                        gz_topic_name="${gz_topic_name}"
+                        image_width="${image_width}"
+                        image_height="${image_height}"
+                        h_fov="${h_fov}"
+                        v_fov="${v_fov}"
+                        triggered="${triggered}"
+                        camera_info_topic="${gz_topic_name}/camera_info"/>
+        <xacro:gazebo_aligned_depth_camera name="${name}"
+                                           fps="${fps}"
+                                           gz_topic_name="${gz_topic_name}"
+                                           image_width="${image_width}"
+                                           image_height="${image_height}"
+                                           fx="${fx}" fy="${fy}" cx="${cx}" cy="${cy}"
+                                           h_fov="${h_fov}"
+                                           v_fov="${v_fov}"
+                                           min_depth="${depth_near_m}"
+                                           max_depth="${depth_far_m}"
+                                           camera_info_topic="${gz_topic_name}/aligned_depth/camera_info"/>
+        <xacro:gazebo_depth_camera name="${name}"
+                                   fps="${fps}"
+                                   gz_topic_name="${gz_topic_name}/native_depth/image"
+                                   image_width="${depth_image_width}"
+                                   image_height="${depth_image_height}"
+                                   fx="${depth_fx}" fy="${depth_fy}" cx="${depth_cx}" cy="${depth_cy}"
+                                   k1="${depth_k1}" k2="${depth_k2}" k3="${depth_k3}" p1="${depth_p1}" p2="${depth_p2}"
+                                   h_fov="${depth_h_fov}"
+                                   v_fov="${depth_v_fov}"
+                                   min_depth="${depth_near_m}"
+                                   max_depth="${depth_far_m}"/>
+    </xacro:if>
 </xacro:macro>
 </robot>

File: src/camera_ws/realsense2_gz_description/urdf/rgb_camera.gazebo.xacro (robot description, xacro)
@@ -21,5 +21,6 @@
   image_height:=720
   h_fov
-  v_fov">
+  v_fov
+  camera_info_topic:=__default__">
     <!--
     Assumptions
@@ -30,4 +31,7 @@
         <sensor name="${name}" type="camera">
             <camera>
+                <xacro:if value="${camera_info_topic != '__default__'}">
+                    <camera_info_topic>${camera_info_topic}</camera_info_topic>
+                </xacro:if>
                 <horizontal_fov>${h_fov}</horizontal_fov>
                 <image>

File: src/myrobot_simulation/config/robots/fairino_arm/fairino_arm_camera_mount.xacro (robot description, xacro)
@@ -8,4 +8,5 @@
     </xacro:camera_v0>
     <xacro:camera_gazebo_v0
+      sensor_type="rgbd"
       fps="${camera_fps}"
       image_width="${camera_image_width}"

File: src/myrobot_simulation/config/robots/fairino_arm/fairino_arm_handeye_camera_mount.xacro (robot description, xacro)
@@ -13,5 +13,5 @@
     </xacro:camera_v0>
     <xacro:camera_gazebo_v0
-      sensor_type="rgb"
+      sensor_type="rgbd"
       fps="${camera_fps}"
       image_width="${camera_image_width}"
