Commit message: graspnet和llm-control优化

File: src/myrobot_simulation/config/robots/fairino_arm/fairino_arm_eye_on_base_gazebo.urdf.xacro (robot description, xacro)
@@ -11,5 +11,5 @@
   <xacro:include filename="fairino_arm_calibration_board.xacro"/>
   <xacro:fairino_arm_calibration_board
-    parent="grasp_frame"
+    parent="tool0"
     xyz="$(arg calibration_board_x) $(arg calibration_board_y) $(arg calibration_board_z)"
     rpy="$(arg calibration_board_roll) $(arg calibration_board_pitch) $(arg calibration_board_yaw)"/>

File: src/myrobot_simulation/config/robots/fairino_arm/fairino_arm_handeye_camera_mount.xacro (robot description, xacro)
@@ -6,7 +6,7 @@
       Gazebo calibration profile uses a clean eye-in-hand visual mount instead
       of replaying a noisy real-world calibration result. The D435 is placed on
-      the -Y side of grasp_frame with the optical axis along grasp_frame +Z.
+      the -Y side of tool0 with the optical axis along tool0 +Z.
     -->
-    <xacro:camera_v0 parent="grasp_frame">
+    <xacro:camera_v0 parent="tool0">
       <origin xyz="0.000 -0.05 -0.09"
               rpy="0 -1.57079632679 -1.57079632679"/>

File: src/myrobot_support/fairino_arm_moveit_descriptions/urdf/fairino_arm_moveit_descriptions.urdf (robot description, URDF)
Before this commit: robot fairino_arm_moveit_descriptions, 11 links, 10 joints
Links:
- removed link grasp_frame
- added link tool0
Joints:
- removed joint wrist3_to_grasp_frame
- added joint wrist3_to_tool0: type fixed, parent wrist3_link, child tool0, origin xyz=0 0 0.2168 rpy=0 0 0
