Commit message: 2026 0824 1720

File: src/myrobot_simulation/config/robots/fairino_arm/fairino_arm_inhand_gazebo.urdf.xacro (robot description, xacro)
@@ -24,8 +24,23 @@
   <xacro:arg name="camera_depth_far_m" default="3.0"/>
   <xacro:include filename="$(find fairino_arm_moveit_descriptions)/urdf/fairino_arm_moveit_descriptions.urdf"/>
+  <xacro:include filename="$(find fairino_arm_moveit_descriptions)/urdf/camera/camera.xacro"/>
+  <xacro:include filename="../common/gazebo_friction.xacro"/>
   <xacro:include filename="../common/gazebo_plugins.xacro"/>
   <xacro:include filename="../common/gazebo_ros2_control.xacro"/>
-  <xacro:include filename="fairino_arm_gripper_friction.xacro"/>
-  <xacro:include filename="fairino_arm_handeye_camera_mount.xacro"/>
+  <xacro:macro name="fairino_arm_gazebo_handeye_camera" params="camera_fps:=30 camera_image_width:=1280 camera_image_height:=720 camera_fx:=0 camera_fy:=0 camera_cx:=0 camera_cy:=0 camera_k1:=0 camera_k2:=0 camera_k3:=0 camera_p1:=0 camera_p2:=0 camera_noise_stddev:=0 camera_h_fov:=1.2042771838760873 camera_v_fov:=0.7330382858376184 camera_depth_image_width:=1280 camera_depth_image_height:=720 camera_depth_fx:=0 camera_depth_fy:=0 camera_depth_cx:=0 camera_depth_cy:=0 camera_depth_k1:=0 camera_depth_k2:=0 camera_depth_k3:=0 camera_depth_p1:=0 camera_depth_p2:=0 camera_depth_h_fov:=1.5184364492350666 camera_depth_v_fov:=1.0122909661567112 camera_depth_near_m:=0.28 camera_depth_far_m:=3.0">
+    <xacro:camera_v0 parent="tool0">
+      <origin xyz="0.000 -0.05 -0.09" rpy="0 -1.57079632679 -1.57079632679"/>
+    </xacro:camera_v0>
+    <xacro:camera_gazebo_v0 sensor_type="rgbd" fps="${camera_fps}"
+      image_width="${camera_image_width}" image_height="${camera_image_height}"
+      fx="${camera_fx}" fy="${camera_fy}" cx="${camera_cx}" cy="${camera_cy}"
+      k1="${camera_k1}" k2="${camera_k2}" k3="${camera_k3}" p1="${camera_p1}" p2="${camera_p2}"
+      noise_stddev="${camera_noise_stddev}" h_fov="${camera_h_fov}" v_fov="${camera_v_fov}"
+      depth_image_width="${camera_depth_image_width}" depth_image_height="${camera_depth_image_height}"
+      depth_fx="${camera_depth_fx}" depth_fy="${camera_depth_fy}" depth_cx="${camera_depth_cx}" depth_cy="${camera_depth_cy}"
+      depth_k1="${camera_depth_k1}" depth_k2="${camera_depth_k2}" depth_k3="${camera_depth_k3}" depth_p1="${camera_depth_p1}" depth_p2="${camera_depth_p2}"
+      depth_h_fov="${camera_depth_h_fov}" depth_v_fov="${camera_depth_v_fov}"
+      depth_near_m="${camera_depth_near_m}" depth_far_m="${camera_depth_far_m}"/>
+  </xacro:macro>
   <xacro:gz_common_plugins controllers_file="$(arg controllers_file)" enable_sensors="$(arg enable_camera)"/>
   <xacro:if value="$(arg enable_camera)">
@@ -45,5 +60,6 @@
       camera_depth_near_m="$(arg camera_depth_near_m)" camera_depth_far_m="$(arg camera_depth_far_m)"/>
   </xacro:if>
-  <xacro:fairino_arm_gripper_friction/>
+  <xacro:gz_link_friction link="finger1" mu1="500.0" mu2="500.0" kp="30000" kd="15"/>
+  <xacro:gz_link_friction link="finger2" mu1="500.0" mu2="500.0" kp="30000" kd="15"/>
   <xacro:gz_six_axis_velocity_control
     name="GazeboSimSystem"

File: src/myrobot_simulation/config/robots/fairino_arm/fairino_arm_onbase_gazebo.urdf.xacro (robot description, xacro)
@@ -24,8 +24,24 @@
   <xacro:arg name="camera_depth_far_m" default="3.0"/>
   <xacro:include filename="$(find fairino_arm_moveit_descriptions)/urdf/fairino_arm_moveit_descriptions.urdf"/>
+  <xacro:include filename="$(find fairino_arm_moveit_descriptions)/urdf/camera/camera.xacro"/>
+  <xacro:include filename="../common/gazebo_friction.xacro"/>
   <xacro:include filename="../common/gazebo_plugins.xacro"/>
   <xacro:include filename="../common/gazebo_ros2_control.xacro"/>
-  <xacro:include filename="fairino_arm_gripper_friction.xacro"/>
-  <xacro:include filename="fairino_arm_camera_mount.xacro"/>
+  <xacro:macro name="fairino_arm_gazebo_camera" params="camera_fps:=60 camera_image_width:=640 camera_image_height:=480 camera_fx:=0 camera_fy:=0 camera_cx:=0 camera_cy:=0 camera_k1:=0 camera_k2:=0 camera_k3:=0 camera_p1:=0 camera_p2:=0 camera_noise_stddev:=0 camera_h_fov:=1.2042771838760873 camera_v_fov:=0.7330382858376184 camera_depth_image_width:=1280 camera_depth_image_height:=720 camera_depth_fx:=0 camera_depth_fy:=0 camera_depth_cx:=0 camera_depth_cy:=0 camera_depth_k1:=0 camera_depth_k2:=0 camera_depth_k3:=0 camera_depth_p1:=0 camera_depth_p2:=0 camera_depth_h_fov:=1.5184364492350666 camera_depth_v_fov:=1.0122909661567112 camera_depth_near_m:=0.28 camera_depth_far_m:=3.0">
+    <xacro:property name="PI" value="3.14159274"/>
+    <xacro:camera_v0 parent="base_link">
+      <origin xyz="0.25 0.7 1.0" rpy="0 ${79*PI/180} ${-PI/2}"/>
+    </xacro:camera_v0>
+    <xacro:camera_gazebo_v0 sensor_type="rgbd" fps="${camera_fps}"
+      image_width="${camera_image_width}" image_height="${camera_image_height}"
+      fx="${camera_fx}" fy="${camera_fy}" cx="${camera_cx}" cy="${camera_cy}"
+      k1="${camera_k1}" k2="${camera_k2}" k3="${camera_k3}" p1="${camera_p1}" p2="${camera_p2}"
+      noise_stddev="${camera_noise_stddev}" h_fov="${camera_h_fov}" v_fov="${camera_v_fov}"
+      depth_image_width="${camera_depth_image_width}" depth_image_height="${camera_depth_image_height}"
+      depth_fx="${camera_depth_fx}" depth_fy="${camera_depth_fy}" depth_cx="${camera_depth_cx}" depth_cy="${camera_depth_cy}"
+      depth_k1="${camera_depth_k1}" depth_k2="${camera_depth_k2}" depth_k3="${camera_depth_k3}" depth_p1="${camera_depth_p1}" depth_p2="${camera_depth_p2}"
+      depth_h_fov="${camera_depth_h_fov}" depth_v_fov="${camera_depth_v_fov}"
+      depth_near_m="${camera_depth_near_m}" depth_far_m="${camera_depth_far_m}"/>
+  </xacro:macro>
   <xacro:gz_common_plugins controllers_file="$(arg controllers_file)" enable_sensors="$(arg enable_camera)"/>
   <xacro:if value="$(arg enable_camera)">
@@ -45,5 +61,6 @@
       camera_depth_near_m="$(arg camera_depth_near_m)" camera_depth_far_m="$(arg camera_depth_far_m)"/>
   </xacro:if>
-  <xacro:fairino_arm_gripper_friction/>
+  <xacro:gz_link_friction link="finger1" mu1="500.0" mu2="500.0" kp="30000" kd="15"/>
+  <xacro:gz_link_friction link="finger2" mu1="500.0" mu2="500.0" kp="30000" kd="15"/>
   <xacro:gz_six_axis_velocity_control
     name="GazeboSimSystem"
