Commit message: 2026 0825 1616-位置伺服仿真和实机版本优化（标定码识别）
Co-authored-by: Copilot <copilot@github.com>

File: src/myrobot_simulation/config/robots/fairino3_v6/fairino3_v6_gazebo.urdf.xacro (robot description, xacro)
@@ -2,11 +2,46 @@
 <robot xmlns:xacro="http://www.ros.org/wiki/xacro" name="fairino3_v6_robot">
   <xacro:arg name="initial_positions_file" default="$(find fairino3_v6_moveit2_config)/config/initial_positions.yaml"/>
-  <xacro:arg name="controllers_file" default="$(find fairino3_v6_moveit2_config)/config/ros2_controllers.yaml"/>
-  <xacro:arg name="enable_camera" default="false"/>
+  <xacro:arg name="controllers_file" default="$(find fairino3_v6_moveit2_config)/config/ros2_controllers_gazebo_velocity.yaml"/>
+  <xacro:arg name="enable_camera" default="true"/>
+  <xacro:arg name="camera_fps" default="60"/>
+  <xacro:arg name="camera_image_width" default="640"/>
+  <xacro:arg name="camera_image_height" default="480"/>
+  <xacro:arg name="camera_fx" default="0"/><xacro:arg name="camera_fy" default="0"/>
+  <xacro:arg name="camera_cx" default="0"/><xacro:arg name="camera_cy" default="0"/>
+  <xacro:arg name="camera_k1" default="0"/><xacro:arg name="camera_k2" default="0"/><xacro:arg name="camera_k3" default="0"/>
+  <xacro:arg name="camera_p1" default="0"/><xacro:arg name="camera_p2" default="0"/><xacro:arg name="camera_noise_stddev" default="0"/>
+  <xacro:arg name="camera_h_fov" default="1.2042771838760873"/>
+  <xacro:arg name="camera_v_fov" default="0.7330382858376184"/>
+  <xacro:arg name="camera_depth_image_width" default="1280"/>
+  <xacro:arg name="camera_depth_image_height" default="720"/>
+  <xacro:arg name="camera_depth_fx" default="0"/><xacro:arg name="camera_depth_fy" default="0"/>
+  <xacro:arg name="camera_depth_cx" default="0"/><xacro:arg name="camera_depth_cy" default="0"/>
+  <xacro:arg name="camera_depth_k1" default="0"/><xacro:arg name="camera_depth_k2" default="0"/><xacro:arg name="camera_depth_k3" default="0"/>
+  <xacro:arg name="camera_depth_p1" default="0"/><xacro:arg name="camera_depth_p2" default="0"/>
+  <xacro:arg name="camera_depth_h_fov" default="1.5184364492350666"/>
+  <xacro:arg name="camera_depth_v_fov" default="1.0122909661567112"/>
+  <xacro:arg name="camera_depth_near_m" default="0.28"/>
+  <xacro:arg name="camera_depth_far_m" default="3.0"/>
   <xacro:include filename="$(find fairino_description)/urdf/fairino3_v6.urdf"/>
+  <xacro:include filename="$(find fairino_arm_moveit_descriptions)/urdf/camera/camera.xacro"/>
   <xacro:include filename="../common/gazebo_plugins.xacro"/>
   <xacro:include filename="../common/gazebo_ros2_control.xacro"/>
-  <xacro:gz_common_plugins controllers_file="$(arg controllers_file)" enable_sensors="false"/>
-  <xacro:gz_six_axis_position_control
+  <xacro:gz_common_plugins controllers_file="$(arg controllers_file)" enable_sensors="$(arg enable_camera)"/>
+  <xacro:if value="$(arg enable_camera)">
+    <xacro:camera_v0 parent="base_link">
+      <origin xyz="0.25 0.7 1.0" rpy="0 ${79*3.14159274/180} ${-3.14159274/2}"/>
+    </xacro:camera_v0>
+    <xacro:camera_gazebo_v0 sensor_type="rgbd" fps="$(arg camera_fps)"
+      image_width="$(arg camera_image_width)" image_height="$(arg camera_image_height)"
+      fx="$(arg camera_fx)" fy="$(arg camera_fy)" cx="$(arg camera_cx)" cy="$(arg camera_cy)"
+      k1="$(arg camera_k1)" k2="$(arg camera_k2)" k3="$(arg camera_k3)" p1="$(arg camera_p1)" p2="$(arg camera_p2)"
+      noise_stddev="$(arg camera_noise_stddev)" h_fov="$(arg camera_h_fov)" v_fov="$(arg camera_v_fov)"
+      depth_image_width="$(arg camera_depth_image_width)" depth_image_height="$(arg camera_depth_image_height)"
+      depth_fx="$(arg camera_depth_fx)" depth_fy="$(arg camera_depth_fy)" depth_cx="$(arg camera_depth_cx)" depth_cy="$(arg camera_depth_cy)"
+      depth_k1="$(arg camera_depth_k1)" depth_k2="$(arg camera_depth_k2)" depth_k3="$(arg camera_depth_k3)" depth_p1="$(arg camera_depth_p1)" depth_p2="$(arg camera_depth_p2)"
+      depth_h_fov="$(arg camera_depth_h_fov)" depth_v_fov="$(arg camera_depth_v_fov)"
+      depth_near_m="$(arg camera_depth_near_m)" depth_far_m="$(arg camera_depth_far_m)"/>
+  </xacro:if>
+  <xacro:gz_six_axis_velocity_control
     name="GazeboSimSystem"
     initial_positions_file="$(arg initial_positions_file)"/>

File: src/myrobot_simulation/config/robots/fairino_arm/fairino_arm_calibration_onbase_gazebo.urdf.xacro (robot description, xacro)
@@ -1,4 +1,4 @@
 <?xml version="1.0"?>
-<robot xmlns:xacro="http://www.ros.org/wiki/xacro" name="fairino_arm">
+<robot xmlns:xacro="http://www.ros.org/wiki/xacro" name="fairino_arm_moveit_descriptions">
   <xacro:arg name="calibration_board_x" default="0.00"/>
   <xacro:arg name="calibration_board_y" default="-0.03"/>

File: src/myrobot_simulation/config/robots/fairino_arm/fairino_arm_inhand_gazebo.urdf.xacro (robot description, xacro)
@@ -1,4 +1,4 @@
 <?xml version="1.0"?>
-<robot xmlns:xacro="http://www.ros.org/wiki/xacro" name="fairino_arm">
+<robot xmlns:xacro="http://www.ros.org/wiki/xacro" name="fairino_arm_moveit_descriptions">
   <xacro:arg name="initial_positions_file" default="$(find fairino_arm_moveit_config)/config/initial_positions.yaml"/>
   <xacro:arg name="controllers_file" default="$(find fairino_arm_moveit_config)/config/ros2_controllers_gazebo_velocity.yaml"/>

File: src/myrobot_simulation/config/robots/fairino_arm/fairino_arm_onbase_gazebo.urdf.xacro (robot description, xacro)
@@ -1,4 +1,4 @@
 <?xml version="1.0"?>
-<robot xmlns:xacro="http://www.ros.org/wiki/xacro" name="fairino_arm">
+<robot xmlns:xacro="http://www.ros.org/wiki/xacro" name="fairino_arm_moveit_descriptions">
   <xacro:arg name="initial_positions_file" default="$(find fairino_arm_moveit_config)/config/initial_positions.yaml"/>
   <xacro:arg name="controllers_file" default="$(find fairino_arm_moveit_config)/config/ros2_controllers_gazebo_velocity.yaml"/>

File: src/myrobot_support/fairino_description/urdf/fairino3_v6.urdf (robot description, URDF)
Before this commit: robot fairino3_v6_robot, 9 links, 8 joints
Joints:
- joint tool0_fixed_joint: origin xyz=0 0 0.1 rpy=0 0 0 -> xyz=0 0 0.2168 rpy=0 0 0
